File: wled_pcb1.kicad_pcb (KiCad board)
At the start: 2 copper layers, 78.7 x 45.7 mm, 10 parts, among them J1 Conn_01x15, J2 conn_esp_left, J3 12v_input, J4 led_output, SW1 SW_SPST, SW2 SW_Push, U1 SN74AHCT125N

Commit message: cleanup and update
Parts:
- removed SW1: SW_SPST, Button_Switch_THT:SW_DIP_SPSTx01_Slide_9.78x4.72mm_W7.62mm_P2.54mm
- added D1: 1N4149, Diode_THT:D_DO-35_SOD27_P7.62mm_Horizontal, F.Cu at (205.7, 120.7)
- added H1: MountingHole_Pad, Connector_Pin:Pin_D1.0mm_L10.0mm, F.Cu at (162.6, 106.7)
- added H2: MountingHole_Pad, Connector_Pin:Pin_D1.0mm_L10.0mm, F.Cu at (162.6, 116.8)
- added JP1: SolderJumper_2_Open, Jumper:SolderJumper-2_P1.3mm_Open_RoundedPad1.0x1.5mm, F.Cu at (162.6, 111.8)
- added REF**: MountingHole_4.3mm_M4_ISO7380, MountingHole:MountingHole_4.3mm_M4_ISO7380, F.Cu at (219.7, 104.1)
- added REF**: MountingHole_4.3mm_M4_ISO7380, MountingHole:MountingHole_4.3mm_M4_ISO7380, F.Cu at (132.1, 104.1)
- added REF**: MountingHole_4.3mm_M4_ISO7380, MountingHole:MountingHole_4.3mm_M4_ISO7380, F.Cu at (219.7, 139.7)
- added REF**: MountingHole_4.3mm_M4_ISO7380, MountingHole:MountingHole_4.3mm_M4_ISO7380, F.Cu at (132.1, 139.7)
- SW2: footprint Button_Switch_THT:SW_DIP_SPSTx01_Piano_10.8x4.1mm_W7.62mm_P2.54mm -> SN75AHCT125N:button_pianoswitch
- moved J3 33.4 mm to (210.8, 104.1), turned to 180 degrees
- moved R1 33.0 mm to (182.9, 116.8), turned to 180 degrees
- moved J4 22.7 mm to (185.4, 104.1), turned to 180 degrees
- moved F1 22.7 mm to (193.0, 104.1)
- moved SW2 16.3 mm to (193.0, 116.8), turned to 180 degrees
- moved PS1 11.4 mm to (191.8, 132.1)
- moved J1 10.2 mm to (167.6, 104.1)
- moved U1 5.24 mm to (146.1, 114.3)
Connections:
- net Net-(J3-Pad2) renamed 12fused
- F1 pad 1: Net-(F1-Pad1) -> +12V
- PS1 pad 2: +12V -> Net-(D1-Pad1)
Routing:
- net GND: track 53.5 -> 7.18 mm, vias 1 -> 2
- net Net-(J4-Pad2): track 91.5 -> 58.0 mm
- net Net-(J1-Pad4): track 44.8 -> 22.4 mm
- net +5V: track 44.8 -> 61.4 mm
- net +12V: track 27.5 -> 17.9 mm
- net Net-(F1-Pad1): track 8.13 -> 0.00 mm
- net 12fused: track 7.48 -> 0.00 mm
- net Net-(J1-Pad5): track 19.9 -> 26.9 mm
- net Net-(D1-Pad1): track 0.00 -> 6.35 mm
- net Net-(J1-Pad6): track 6.13 -> 5.08 mm
- added copper zone on F.Cu, net +12V
- added copper zone on F.Cu, net 12fused
Other:
- board size 78.7 x 45.7 mm -> 99.1 x 45.7 mm

Commit message: printable?
Parts:
- R1: value R -> 10K
- moved R1 9.16 mm to (175.3, 111.8), turned to -90 degrees
Routing:
- net Net-(J1-Pad6): track 5.08 -> 11.2 mm
- net GND: track 7.18 -> 12.3 mm
Other:
- board text added: "12V"
- board text added: "D"
- board text added: "ESP8266"
- board text added: "GND"
- board text added: "Lennart & Jochem"
- board text added: "left"
- board text added: "right"
- board text added: "wled_v2"
