File: wled_pcb1.kicad_sch (KiCad schematic)
At the start: 10 parts, among them J1 Conn_01x15, J2 conn_esp_left, J3 12v_input, J4 led_output, SW1 SW_SPST, SW2 SW_Push, U1 SN74AHCT125N

Commit message: cleanup and update
Parts:
- removed SW1: SW_SPST, Button_Switch_THT:SW_DIP_SPSTx01_Slide_9.78x4.72mm_W7.62mm_P2.54mm, symbol Switch:SW_SPST
- added D1: 1N4149, Diode_THT:D_DO-35_SOD27_P7.62mm_Horizontal, symbol Diode:1N4149
- added H1, H2: MountingHole_Pad, Connector_Pin:Pin_D1.0mm_L10.0mm, symbol Mechanical:MountingHole_Pad
- added JP1: SolderJumper_2_Open, Jumper:SolderJumper-2_P1.3mm_Open_RoundedPad1.0x1.5mm, symbol Jumper:SolderJumper_2_Open
- SW2: footprint Button_Switch_THT:SW_DIP_SPSTx01_Piano_10.8x4.1mm_W7.62mm_P2.54mm -> SN75AHCT125N:button_pianoswitch
Connections:
- net +12V: now also F1.1, D1.2 (A); no longer PS1.2 (+Vin)
- net at J1.5 (Pin_5), U1.2 (1A): now also H2.1, JP1.1 (A)
- net at J4.2 (Pin_2), U1.3 (1Y): now also H1.1, JP1.2 (B)
- net 12fused: now reaches F1.2, J3.2 (Pin_2)
- new net: D1.1 (K), PS1.2 (+Vin)
Other:
- moved on the sheet: F1, PS1

Commit message: printable?
Parts:
- R1: value R -> 10K
Changed lines of the file:
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@@
       (effects (font (size 1.27 1.27)) (justify left))
     )
-    (property "Value" "R" (id 1) (at 114.3 57.1499 0)
+    (property "Value" "10K" (id 1) (at 114.3 57.1499 0)
       (effects (font (size 1.27 1.27)) (justify left))
     )
@@
     )
     (path "/584c482d-1251-462e-825c-3a0578bafc6d"
-      (reference "R1") (unit 1) (value "R") (footprint "Resistor_THT:R_Axial_DIN0207_L6.3mm_D2.5mm_P10.16mm_Horizontal")
+      (reference "R1") (unit 1) (value "10K") (footprint "Resistor_THT:R_Axial_DIN0207_L6.3mm_D2.5mm_P10.16mm_Horizontal")
     )
     (path "/6be776b9-ebd1-4fb3-a15a-501f1a1df113"
